File: hardware/uPIC46/uPIC46.kicad_pcb (KiCad board)
At the start: 2 copper layers, 66.6 x 41.3 mm, 96 parts, among them J1 USB_C_Receptacle_USB2.0_16P, J2 Conn_01x14_Socket, J3 Conn_PIC_ICSP_ICD, J4 Conn_01x06_Socket, J5 Screw_Terminal_01x02, J6 Conn_01x06_Socket, J8 Screw_Terminal_01x02, SW1 SW_Push, U1 TPD2E2U06DCK, U2 PIC18F46K22-I/PT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

Commit message: designators
Routing:
- net 3VP: track 271.6 -> 281.1 mm
- net Net-(FB1-Pad2): track 1.80 -> 7.91 mm, vias 0 -> 2
- net D+: track 6.93 -> 12.1 mm
- net D-: track 6.93 -> 11.1 mm, vias 0 -> 2
- net MCLR: track 75.3 -> 79.0 mm
- net PGC: track 19.0 -> 20.8 mm
- net PGD: track 18.5 -> 20.3 mm
- net RE1: track 26.1 -> 27.4 mm
- net PB0: track 24.5 -> 25.8 mm
- net RD5: track 17.6 -> 18.9 mm
- net RE2: track 26.5 -> 27.8 mm
- net RE0: track 24.9 -> 26.2 mm
- net RA4: track 26.4 -> 27.7 mm
- net PB2: track 24.7 -> 26.0 mm
- net PB1: track 24.5 -> 25.8 mm
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- added copper zone on F.Cu, net GND
Other:
- board text added: "3V3P"
- board text added: "A1"
- board text added: "A2"
- board text added: "A3"
- board text added: "A4"
- board text added: "A5"
- board text added: "B0"
- board text added: "B1"
- board text added: "B2"
- board text added: "C1"
- board text added: "C2"
- board text added: "C5"
- board text added: "D4"
- board text added: "D5"
- board text added: "E0"
- board text added: "E1"
- board text added: "E2"
- board text added: "GC"
- board text added: "GD"
- board text added: "GND"
- board text added: "NC"
- board text added: "VBUS"

Commit message: v0
Parts:
- added FID1: Fiducial, Fiducial:Fiducial_1mm_Mask2mm, F.Cu at (121.7, 110.2)
- added FID2: Fiducial, Fiducial:Fiducial_1mm_Mask2mm, F.Cu at (177.3, 98.0)
- added FID3: Fiducial, Fiducial:Fiducial_1mm_Mask2mm, B.Cu at (123.5, 109.0)
- added FID4: Fiducial, Fiducial:Fiducial_1mm_Mask2mm, B.Cu at (147.1, 94.2)
- added REF**: ESD-Logo_6.6x6mm_SilkScreen, Symbol:ESD-Logo_6.6x6mm_SilkScreen, F.Cu at (172.2, 93.7)
- added REF**: WEEE-Logo_4.2x6mm_SilkScreen, Symbol:WEEE-Logo_4.2x6mm_SilkScreen, F.Cu at (144.8, 87.5)
- added REF**: KiCad-Logo2_5mm_SilkScreen, Symbol:KiCad-Logo2_5mm_SilkScreen, B.Cu at (133.8, 81.3)
- moved J5 0.99 mm to (179.8, 109.5)
- moved C9 0.70 mm to (178.8, 90.9)
Routing:
- net VBUS: track 78.4 -> 94.1 mm
- net GND: track 12.5 -> 10.6 mm, vias 79 -> 83
- net /R+: track 20.8 -> 19.4 mm
- net 3VP: track 281.1 -> 281.2 mm, vias 14 -> 23
Other:
- board text added: "0"
- board text added: "0 mm"
- board text added: "0.0000 mm / 0.0000 mm"
- board text added: "0.01 mm"
- board text added: "0.02"
- board text added: "0.035 mm"
- board text added: "0.2000 mm"
- board text added: "0x4D455254"
- board text added: "1"
- board text added: "1.51 mm"
- board text added: "1.6000 mm"
- board text added: "2"
- board text added: "3.3"
- board text added: "4.5"
- board text added: "66.6200 mm x 41.3100 mm"
- board text added: "A"
- board text added: "B"
- board text added: "B.Cu"
- board text added: "B.Mask"
- board text added: "B.Paste"
- board text added: "B.Silkscreen"
- board text added: "BOARD CHARACTERISTICS"
- board text added: "Board Thickness:"
- board text added: "Board overall dimensions:"
- board text added: "Bottom Silk Screen"
- board text added: "Bottom Solder Mask"
- board text added: "Bottom Solder Paste"
- board text added: "CAN Bus"
- board text added: "CANH"
- board text added: "CANL"
- board text added: "Castellated pads:"
- board text added: "Color"
- board text added: "Copper Finish:"
- board text added: "Copper Layer Count:"
- board text added: "Dielectric"
- board text added: "Edge card connectors:"
- board text added: "Epsilon R"
- board text added: "F.Cu"
- board text added: "F.Mask"
- board text added: "F.Paste"
- board text added: "F.Silkscreen"
- board text added: "FR4"
- board text added: "Impedance Control:"
- board text added: "Layer Name"
- board text added: "Loss Tangent"
- board text added: "Material"
- board text added: "Min hole diameter:"
- board text added: "Min track/spacing:"
- board text added: "No"
- board text added: "None"
- board text added: "Not specified"
- board text added: "PIC18F46K22"
- board text added: "Plated Board Edge:"
- board text added: "RS-485"
- board text added: "RST"
- board text added: "Red"
- board text added: "Thickness (mm)"
- board text added: "Top Silk Screen"
- board text added: "Top Solder Mask"
- board text added: "Top Solder Paste"
- board text added: "Type"
- board text added: "White"
- board text added: "copper"
- board text added: "core"
- board text added: "uPIC46"

Commit message: v0
Parts:
- added ?: , , F.Cu at (126.7, 84.9)
- added ?: , , F.Cu at (124.2, 84.9)
- added ?: , , F.Cu at (122.7, 84.9)
- added ?: , , F.Cu at (123.3, 89.0)
- added ?: , , F.Cu at (122.0, 89.0)
- added ?: , , F.Cu at (122.7, 89.9)
- added ?: , , F.Cu at (122.0, 90.8)
- added ?: , , F.Cu at (123.3, 90.8)
- added ?: , , F.Cu at (125.5, 84.9)
Routing:
- net 3VP: vias 23 -> 14

Commit message: v0
Parts:
- removed FID4: Fiducial, Fiducial:Fiducial_1mm_Mask2mm
- FID1, FID2, FID3: footprint Fiducial:Fiducial_1mm_Mask2mm -> Fiducial:Fiducial_0.5mm_Mask1.5mm
- moved FID3 2.42 mm to (121.1, 109.0)
- moved FID2 1.42 mm to (177.7, 99.4)
- moved FID1 1.09 mm to (121.2, 109.1)
- moved J3 0.30 mm to (182.6, 86.1)
Routing:
- net D+: track 12.1 -> 13.1 mm
- net D-: track 11.1 -> 12.1 mm
