File: hardware/uPIC46/uPIC46.kicad_sch (KiCad schematic)
At the start: 96 parts, among them J1 USB_C_Receptacle_USB2.0_16P, J2 Conn_01x14_Socket, J3 Conn_PIC_ICSP_ICD, J4 Conn_01x06_Socket, J5 Screw_Terminal_01x02, J6 Conn_01x06_Socket, J8 Screw_Terminal_01x02, SW1 SW_Push, U1 TPD2E2U06DCK, U2 PIC18F46K22-I/PT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

Commit message: v0
Parts:
- added FID1, FID2, FID3, FID4: Fiducial, Fiducial:Fiducial_1mm_Mask2mm, symbol Mechanical:Fiducial
Other:
- moved on the sheet: J6

Commit message: v0
Parts:
- removed FID4: Fiducial, Fiducial:Fiducial_1mm_Mask2mm, symbol Mechanical:Fiducial
- FID1, FID2, FID3: footprint Fiducial:Fiducial_1mm_Mask2mm -> Fiducial:Fiducial_0.5mm_Mask1.5mm
Changed lines of the file:
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@@
 	)
 	(symbol
-		(lib_id "Mechanical:Fiducial")
-		(at 347.98 227.33 0)
-		(unit 1)
-		(exclude_from_sim no)
-		(in_bom no)
-		(on_board yes)
-		(dnp no)
-		(fields_autoplaced yes)
-		(property "Reference" "FID3"
-			(at 350.52 226.0599 0)
-			(effects
-				(font
-					(size 1.27 1.27)
-				)
-				(justify left)
-			)
-		)
-		(property "Value" "Fiducial"
-			(at 350.52 228.5999 0)
-			(effects
-				(font
-					(size 1.27 1.27)
-				)
-				(justify left)
-			)
-		)
-		(property "Footprint" "Fiducial:Fiducial_1mm_Mask2mm"
-			(at 347.98 227.33 0)
-			(effects
-				(font
-					(size 1.27 1.27)
-				)
-				(hide yes)
-			)
-		)
-		(property "Datasheet" "~"
-			(at 347.98 227.33 0)
-			(effects
-				(font
-					(size 1.27 1.27)
-				)
-				(hide yes)
-			)
-		)
-		(property "Description" "Fiducial Marker"
-			(at 347.98 227.33 0)
-			(effects
-				(font
-					(size 1.27 1.27)
-				)
-				(hide yes)
-			)
-		)
-		(instances
-			(project "uPIC46"
-				(path "/ae565447-02b0-45a3-be14-51df2894d4d2"
-					(reference "FID3")
-					(unit 1)
-				)
-			)
-		)
-	)
-	(symbol
 		(lib_id "power:GND")
 		(at 363.22 82.55 0)
@@
 	)
 	(symbol
-		(lib_id "Device:C")
-		(at 24.13 129.54 0)
+		(lib_id "Mechanical:Fiducial")
+		(at 359.41 218.44 0)
 		(unit 1)
 		(exclude_from_sim no)
-		(in_bom yes)
+		(in_bom no)
 		(on_board yes)
 		(dnp no)
 		(fields_autoplaced yes)
-		(property "Reference" "C16"
-			(at 27.94 128.2699 0)
+		(property "Reference" "FID2"
+			(at 361.95 217.1699 0)
 			(effects
 				(font
@@
 			)
 		)
-		(property "Value" "10uF"
-			(at 27.94 130.8099 0)
+		(property "Value" "Fiducial"
+			(at 361.95 219.7099 0)
 			(effects
 				(font
@@
 			)
 		)
-		(property "Footprint" "Capacitor_SMD:C_1206_3216Metric"
-			(at 25.0952 133.35 0)
+		(property "Footprint" "Fiducial:Fiducial_0.5mm_Mask1.5mm"
+			(at 359.41 218.44 0)
 			(effects
 				(font
@@
 		)
 		(property "Datasheet" "~"
-			(at 24.13 129.54 0)
+			(at 359.41 218.44 0)
 			(effects
 				(font
@@
 			)
 		)
-		(property "Description" "Unpolarized capacitor"
-			(at 24.13 129.54 0)
+		(property "Description" "Fiducial Marker"
+			(at 359.41 218.44 0)
 			(effects
 				(font
@@
 			)
 		)
-		(pin "1"
-		)
-		(pin "2"
-		)
 		(instances
-			(project ""
+			(project "uPIC46"
 				(path "/ae565447-02b0-45a3-be14-51df2894d4d2"
-					(reference "C16")
+					(reference "FID2")
 					(unit 1)
 				)
@@
 	)
 	(symbol
-		(lib_id "Mechanical:Fiducial")
-		(at 370.84 214.63 0)
+		(lib_id "Device:C")
+		(at 24.13 129.54 0)
 		(unit 1)
 		(exclude_from_sim no)
-		(in_bom no)
+		(in_bom yes)
 		(on_board yes)
 		(dnp no)
 		(fields_autoplaced yes)
-		(property "Reference" "FID2"
-			(at 373.38 213.3599 0)
+		(property "Reference" "C16"
+			(at 27.94 128.2699 0)
 			(effects
 				(font
@@
 			)
 		)
-		(property "Value" "Fiducial"
-			(at 373.38 215.8999 0)
+		(property "Value" "10uF"
+			(at 27.94 130.8099 0)
 			(effects
 				(font
@@
 			)
 		)
-		(property "Footprint" "Fiducial:Fiducial_1mm_Mask2mm"
-			(at 370.84 214.63 0)
+		(property "Footprint" "Capacitor_SMD:C_1206_3216Metric"
+			(at 25.0952 133.35 0)
 			(effects
 				(font
@@
 		)
 		(property "Datasheet" "~"
-			(at 370.84 214.63 0)
+			(at 24.13 129.54 0)
 			(effects
 				(font
@@
 			)
 		)
-		(property "Description" "Fiducial Marker"
-			(at 370.84 214.63 0)
+		(property "Description" "Unpolarized capacitor"
+			(at 24.13 129.54 0)
 			(effects
 				(font
@@
 			)
 		)
+		(pin "1"
+		)
+		(pin "2"
+		)
 		(instances
-			(project "uPIC46"
+			(project ""
 				(path "/ae565447-02b0-45a3-be14-51df2894d4d2"
-					(reference "FID2")
+					(reference "C16")
 					(unit 1)
 				)
@@
 	)
 	(symbol
-		(lib_id "Mechanical:Fiducial")
-		(at 347.98 214.63 0)
-		(unit 1)
-		(exclude_from_sim no)
-		(in_bom no)
-		(on_board yes)
-		(dnp no)
-		(fields_autoplaced yes)
-		(property "Reference" "FID1"
-			(at 350.52 213.3599 0)
-			(effects
-				(font
-					(size 1.27 1.27)
-				)
-				(justify left)
-			)
-		)
-		(property "Value" "Fiducial"
-			(at 350.52 215.8999 0)
-			(effects
-				(font
-					(size 1.27 1.27)
-				)
-				(justify left)
-			)
-		)
-		(property "Footprint" "Fiducial:Fiducial_1mm_Mask2mm"
-			(at 347.98 214.63 0)
-			(effects
-				(font
-					(size 1.27 1.27)
-				)
-				(hide yes)
-			)
-		)
-		(property "Datasheet" "~"
-			(at 347.98 214.63 0)
-			(effects
-				(font
-					(size 1.27 1.27)
-				)
-				(hide yes)
-			)
-		)
-		(property "Description" "Fiducial Marker"
-			(at 347.98 214.63 0)
-			(effects
-				(font
-					(size 1.27 1.27)
-				)
-				(hide yes)
-			)
-		)
-		(instances
-			(project ""
-				(path "/ae565447-02b0-45a3-be14-51df2894d4d2"
-					(reference "FID1")
-					(unit 1)
-				)
-			)
-		)
-	)
-	(symbol
 		(lib_id "Device:FerriteBead")
 		(at 68.58 30.48 270)
@@
 	)
 	(symbol
+		(lib_id "Mechanical:Fiducial")
+		(at 342.9 218.44 0)
+		(unit 1)
+		(exclude_from_sim no)
+		(in_bom no)
+		(on_board yes)
+		(dnp no)
+		(fields_autoplaced yes)
+		(property "Reference" "FID1"
+			(at 345.44 217.1699 0)
+			(effects
+				(font
+					(size 1.27 1.27)
+				)
+				(justify left)
+			)
+		)
+		(property "Value" "Fiducial"
+			(at 345.44 219.7099 0)
+			(effects
+				(font
+					(size 1.27 1.27)
+				)
+				(justify left)
+			)
+		)
+		(property "Footprint" "Fiducial:Fiducial_0.5mm_Mask1.5mm"
+			(at 342.9 218.44 0)
+			(effects
+				(font
+					(size 1.27 1.27)
+				)
+				(hide yes)
+			)
+		)
+		(property "Datasheet" "~"
+			(at 342.9 218.44 0)
+			(effects
+				(font
+					(size 1.27 1.27)
+				)
+				(hide yes)
+			)
+		)
+		(property "Description" "Fiducial Marker"
+			(at 342.9 218.44 0)
+			(effects
+				(font
+					(size 1.27 1.27)
+				)
+				(hide yes)
+			)
+		)
+		(instances
+			(project ""
+				(path "/ae565447-02b0-45a3-be14-51df2894d4d2"
+					(reference "FID1")
+					(unit 1)
+				)
+			)
+		)
+	)
+	(symbol
 		(lib_id "power:VBUS")
 		(at 185.42 27.94 0)
@@
 	)
 	(symbol
+		(lib_id "Mechanical:Fiducial")
+		(at 374.65 218.44 0)
+		(unit 1)
+		(exclude_from_sim no)
+		(in_bom no)
+		(on_board yes)
+		(dnp no)
+		(fields_autoplaced yes)
+		(property "Reference" "FID3"
+			(at 377.19 217.1699 0)
+			(effects
+				(font
+					(size 1.27 1.27)
+				)
+				(justify left)
+			)
+		)
+		(property "Value" "Fiducial"
+			(at 377.19 219.7099 0)
+			(effects
+				(font
+					(size 1.27 1.27)
+				)
+				(justify left)
+			)
+		)
+		(property "Footprint" "Fiducial:Fiducial_0.5mm_Mask1.5mm"
+			(at 374.65 218.44 0)
+			(effects
+				(font
+					(size 1.27 1.27)
+				)
+				(hide yes)
+			)
+		)
+		(property "Datasheet" "~"
+			(at 374.65 218.44 0)
+			(effects
+				(font
+					(size 1.27 1.27)
+				)
+				(hide yes)
+			)
+		)
+		(property "Description" "Fiducial Marker"
+			(at 374.65 218.44 0)
+			(effects
+				(font
+					(size 1.27 1.27)
+				)
+				(hide yes)
+			)
+		)
+		(instances
+			(project "uPIC46"
+				(path "/ae565447-02b0-45a3-be14-51df2894d4d2"
+					(reference "FID3")
+					(unit 1)
+				)
+			)
+		)
+	)
+	(symbol
 		(lib_id "Device:R")
 		(at 297.18 214.63 180)
@@
 					(unit 1)
 				)
-			)
-		)
-	)
-	(symbol
-		(lib_id "Mechanical:Fiducial")
-		(at 370.84 228.6 0)
-		(unit 1)
-		(exclude_from_sim no)
-		(in_bom no)
-		(on_board yes)
-		(dnp no)
-		(fields_autoplaced yes)
-		(property "Reference" "FID4"
-			(at 373.38 227.3299 0)
-			(effects
-				(font
-					(size 1.27 1.27)
-				)
-				(justify left)
-			)
-		)
-		(property "Value" "Fiducial"
-			(at 373.38 229.8699 0)
-			(effects
-				(font
-					(size 1.27 1.27)
-				)
-				(justify left)
-			)
-		)
-		(property "Footprint" "Fiducial:Fiducial_1mm_Mask2mm"
-			(at 370.84 228.6 0)
-			(effects
-				(font
-					(size 1.27 1.27)
-				)
-				(hide yes)
-			)
-		)
-		(property "Datasheet" "~"
-			(at 370.84 228.6 0)
-			(effects
-				(font
-					(size 1.27 1.27)
-				)
-				(hide yes)
-			)
-		)
-		(property "Description" "Fiducial Marker"
-			(at 370.84 228.6 0)
-			(effects
-				(font
-					(size 1.27 1.27)
-				)
-				(hide yes)
-			)
-		)
-		(instances
-			(project "uPIC46"
-				(path "/ae565447-02b0-45a3-be14-51df2894d4d2"
-					(reference "FID4")
-					(unit 1)
-				)
